File: CAD/Eagle/FindMeSAT_MB_1V1.sch (EAGLE design)
At the start: 131 parts, among them J291 MCX-J-P-X-RA-SM1, J685 SMA_CON, J701 MOLEX_105017-0001, J801 MICROSIM-8P_SDCARD-8P_MOLEX-1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, J901 JST_S3B-XH-A, Q101 ABS07-32.768KHZ, Q651 ABM3B-16MHZ-10-R50-1-U, U1001 CFPT-141-20MHZ, U101 ATXMEGA256A3BU-AU, U1011 OPA354, U1021 OPA354, U1111 LM2831YMF, U1121 LM4120IM5-3.0, U201 SIM808, U301 MPU-9250, U401 MS5607-02BA03, U501 SHT31-DIS, U601 AX5243

Commit message: CAD - multiple corrections of V1.1 redesign findings list
Parts:
- added FM1201, FM1202, FM1203, FM1204: FIDUCIAL_MARK_1MM, df4iah_fiducial:FIDUCIAL_MARK_1MM
- Q651: device adafruit:CRYSTALCTS406 -> df4iah_crystal:ABM03B-16.000MHZ
Connections:
- net GND: now also Q651.3
Changed lines of the file:
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@@
 <part name="GND611" library="df4iah_supply" deviceset="GND" device=""/>
 <part name="GND612" library="df4iah_supply" deviceset="GND" device=""/>
-<part name="Q651" library="adafruit" deviceset="CRYSTAL" device="CTS406" value="ABM3B-16MHZ-10-R50-1-U"/>
+<part name="Q651" library="df4iah_crystal" deviceset="ABM03B-16.000MHZ" device="" value="ABM3B-16MHZ-10-R50-1-U"/>
 <part name="L671" library="rcl" deviceset="R-EU_" device="R0603" value="22nH"/>
 <part name="C681" library="rcl" deviceset="C-EU" device="C0603" value="68pF"/>
@@
 <part name="R301" library="rcl" deviceset="R-EU_" device="R0603" value="68R"/>
 <part name="JP201" library="df4iah_connector" deviceset="HEADER-1X2" device="" value="POW"/>
+<part name="FM1201" library="df4iah_fiducial" deviceset="FIDUCIAL_MARK_1MM" device=""/>
+<part name="FM1202" library="df4iah_fiducial" deviceset="FIDUCIAL_MARK_1MM" device=""/>
+<part name="FM1203" library="df4iah_fiducial" deviceset="FIDUCIAL_MARK_1MM" device=""/>
+<part name="FM1204" library="df4iah_fiducial" deviceset="FIDUCIAL_MARK_1MM" device=""/>
+<part name="GND651" library="df4iah_supply" deviceset="GND" device=""/>
 </parts>
 <sheets>
@@
 <instance part="J685" gate="A" x="228.6" y="86.36"/>
 <instance part="GND689" gate="1" x="226.06" y="63.5"/>
+<instance part="GND651" gate="1" x="137.16" y="127"/>
 </instances>
 <busses>
@@
 <pinref part="J685" gate="A" pin="2"/>
 <wire x1="226.06" y1="66.04" x2="226.06" y2="76.2" width="0.1524" layer="91"/>
+</segment>
+<segment>
+<pinref part="Q651" gate="G$1" pin="3"/>
+<pinref part="GND651" gate="1" pin="GND"/>
 </segment>
 </net>
@@
 <segment>
 <pinref part="U601" gate="A" pin="CLK16N"/>
-<wire x1="116.84" y1="129.54" x2="144.78" y2="129.54" width="0.1524" layer="91"/>
-<wire x1="144.78" y1="129.54" x2="144.78" y2="134.62" width="0.1524" layer="91"/>
+<wire x1="116.84" y1="129.54" x2="129.286" y2="129.54" width="0.1524" layer="91"/>
+<wire x1="129.286" y1="129.54" x2="129.54" y2="121.92" width="0.1524" layer="91"/>
+<wire x1="129.54" y1="121.92" x2="144.78" y2="121.92" width="0.1524" layer="91"/>
+<wire x1="144.78" y1="121.92" x2="144.78" y2="134.62" width="0.1524" layer="91"/>
 <pinref part="Q651" gate="G$1" pin="2"/>
 <wire x1="144.78" y1="134.62" x2="139.7" y2="134.62" width="0.1524" layer="91"/>
@@
 <instance part="GND1201" gate="1" x="58.42" y="129.54"/>
 <instance part="GND1203" gate="1" x="172.72" y="50.8"/>
+<instance part="FM1201" gate="G$1" x="63.5" y="121.92"/>
+<instance part="FM1202" gate="G$1" x="63.5" y="63.5"/>
+<instance part="FM1203" gate="G$1" x="177.8" y="63.5"/>
+<instance part="FM1204" gate="G$1" x="177.8" y="121.92"/>
 </instances>
 <busses>

Commit message: CAD - first round of V1.0 --> V1.1 redesign done
Parts:
- renumbered J291 to X291, J685 to X685, J701 to X701, J801 to X801, J901 to X901, JP111 to X111, JP121 to X121, JP131 to X131, JP181 to X181

Commit message: CAD/Docs - V1.1 candidate created
Parts:
- X121: value HEADER-2X3 -> MOLEX_90130_2X03; device df4iah_connector:HEADER-2X3 -> df4iah_connector:MOLEX_90130_2X03
Connections:
- net +3V3: now also X121.6; no longer X121.5
- net +5V: now also X121.4; no longer X121.3
- net GND: now also X121.2, X121.5; no longer X121.1, X121.6
- net SCL2: now also X121.1; no longer X121.2
- net SDA2: now also X121.3; no longer X121.4
Changed lines of the file:
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@@
 <part name="R132" library="rcl" deviceset="R-EU_" device="R0603" value="68R"/>
 <part name="R112" library="rcl" deviceset="R-EU_" device="R0603" value="10kR"/>
-<part name="X131" library="df4iah_connector" deviceset="HEADER-2X3" device="" value=""/>
+<part name="X131" library="df4iah_connector" deviceset="HEADER-2X3" device="" value="HEADER-2X3"/>
 <part name="GND131" library="df4iah_supply" deviceset="GND" device=""/>
 <part name="R1002" library="rcl" deviceset="R-EU_" device="R0603" value="10kR"/>
-<part name="X111" library="df4iah_connector" deviceset="AVR-JTAG-10" device="" value=""/>
+<part name="X111" library="df4iah_connector" deviceset="AVR-JTAG-10" device="" value="AVR-JTAG-10"/>
 <part name="GND111" library="df4iah_supply" deviceset="GND" device=""/>
 <part name="R111" library="rcl" deviceset="R-EU_" device="R0805" value="0R"/>
@@
 <part name="C141" library="rcl" deviceset="C-EU" device="C0603" value="100pF"/>
 <part name="GND141" library="df4iah_supply" deviceset="GND" device=""/>
-<part name="X121" library="df4iah_connector" deviceset="HEADER-2X3" device="" value=""/>
+<part name="X121" library="df4iah_connector" deviceset="MOLEX_90130_2X03" device="" value="MOLEX_90130_2X03"/>
 <part name="GND121" library="df4iah_supply" deviceset="GND" device=""/>
 <part name="+5V1" library="df4iah_supply" deviceset="+5V" device=""/>
@@
 <part name="X685" library="df4iah_connector" deviceset="SMA_SMT_AMPHENOL-901-143" device="" value="SMA_CON"/>
 <part name="GND689" library="df4iah_supply" deviceset="GND" device=""/>
-<part name="X181" library="df4iah_connector" deviceset="HEADER-2X3" device="" value=""/>
+<part name="X181" library="df4iah_connector" deviceset="HEADER-2X3" device="" value="HEADER-2X3"/>
 <part name="GND181" library="df4iah_supply" deviceset="GND" device=""/>
 <part name="U401" library="df4iah_sensors" deviceset="MS5607-02BA" device="" technology="03"/>
@@
 <pinref part="GND121" gate="1" pin="GND"/>
 <wire x1="50.8" y1="68.58" x2="50.8" y2="76.2" width="0.1524" layer="91"/>
-<pinref part="X121" gate="G$1" pin="6"/>
+<pinref part="X121" gate="G$1" pin="5"/>
 <wire x1="50.8" y1="76.2" x2="48.26" y2="76.2" width="0.1524" layer="91"/>
 <wire x1="50.8" y1="68.58" x2="35.56" y2="68.58" width="0.1524" layer="91"/>
 <wire x1="35.56" y1="68.58" x2="35.56" y2="81.28" width="0.1524" layer="91"/>
-<pinref part="X121" gate="G$1" pin="1"/>
+<pinref part="X121" gate="G$1" pin="2"/>
 <wire x1="35.56" y1="81.28" x2="38.1" y2="81.28" width="0.1524" layer="91"/>
 <junction x="50.8" y="68.58"/>
@@
 <wire x1="55.88" y1="60.96" x2="33.02" y2="60.96" width="0.1524" layer="91"/>
 <wire x1="33.02" y1="60.96" x2="33.02" y2="76.2" width="0.1524" layer="91"/>
-<pinref part="X121" gate="G$1" pin="5"/>
+<pinref part="X121" gate="G$1" pin="6"/>
 <wire x1="33.02" y1="76.2" x2="38.1" y2="76.2" width="0.1524" layer="91"/>
 <junction x="55.88" y="60.96"/>
@@
 <label x="78.74" y="93.98" size="1.778" layer="95"/>
 <wire x1="53.34" y1="93.98" x2="53.34" y2="78.74" width="0.1524" layer="91"/>
-<pinref part="X121" gate="G$1" pin="4"/>
+<pinref part="X121" gate="G$1" pin="3"/>
 <wire x1="53.34" y1="78.74" x2="48.26" y2="78.74" width="0.1524" layer="91"/>
 </segment>
@@
 <label x="78.74" y="91.44" size="1.778" layer="95"/>
 <wire x1="50.8" y1="91.44" x2="50.8" y2="81.28" width="0.1524" layer="91"/>
-<pinref part="X121" gate="G$1" pin="2"/>
+<pinref part="X121" gate="G$1" pin="1"/>
 <wire x1="50.8" y1="81.28" x2="48.26" y2="81.28" width="0.1524" layer="91"/>
 </segment>
@@
 <pinref part="+5V1" gate="G$1" pin="+5V"/>
 <wire x1="25.4" y1="83.82" x2="25.4" y2="78.74" width="0.1524" layer="91"/>
-<pinref part="X121" gate="G$1" pin="3"/>
+<pinref part="X121" gate="G$1" pin="4"/>
 <wire x1="25.4" y1="78.74" x2="38.1" y2="78.74" width="0.1524" layer="91"/>
 </segment>
