File: CAD/Eagle/FindMeSAT_MB_1V2.brd (EAGLE design)
At the start: 99 x 49.2 mm, 135 parts, among them Q101 ABS07-32.768KHZ, Q651 ABM3B-16MHZ-10-R50-1-U, U1001 CFPT-141-20MHZ, U101 ATXMEGA256A3BU-AU, U1011 OPA354, U1021 OPA354, U1111 LM2831YMF, U1121 LM4120IM5-3.0, U201 SIM808, U301 MPU-9250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

Commit message: HW_V1.2 - LCD connector swapped
Connections:
- net +3V3: now also X121.5; no longer X121.6
- net +5V: now also X121.3; no longer X121.4
- net GND: now also X121.1, X121.6; no longer X121.2, X121.5
- net SCL2: now also X121.2; no longer X121.1
- net SDA2: now also X121.4; no longer X121.3
Changed lines of the file:
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@@
 <setting verticaltext="up"/>
 </settings>
-<grid distance="1.27" unitdist="mm" unit="mm" style="lines" multiple="1" display="yes" altdistance="0.127" altunitdist="mm" altunit="mm"/>
+<grid distance="1.27" unitdist="mm" unit="mm" style="lines" multiple="1" display="yes" altdistance="0.003125" altunitdist="mic" altunit="mm"/>
 <layers>
 <layer number="1" name="Top" color="4" fill="1" visible="yes" active="yes"/>
 <layer number="2" name="Route2" color="13" fill="1" visible="yes" active="yes"/>
-<layer number="3" name="Route3" color="4" fill="3" visible="no" active="yes"/>
-<layer number="14" name="Route14" color="1" fill="6" visible="no" active="yes"/>
 <layer number="15" name="Route15" color="11" fill="1" visible="yes" active="yes"/>
 <layer number="16" name="Bottom" color="1" fill="1" visible="yes" active="yes"/>
@@
 <layer number="29" name="tStop" color="7" fill="3" visible="yes" active="yes"/>
 <layer number="30" name="bStop" color="7" fill="6" visible="yes" active="yes"/>
-<layer number="31" name="tCream" color="7" fill="4" visible="yes" active="yes"/>
-<layer number="32" name="bCream" color="7" fill="5" visible="yes" active="yes"/>
+<layer number="31" name="tCream" color="7" fill="4" visible="no" active="yes"/>
+<layer number="32" name="bCream" color="7" fill="5" visible="no" active="yes"/>
 <layer number="33" name="tFinish" color="6" fill="3" visible="no" active="yes"/>
 <layer number="34" name="bFinish" color="6" fill="6" visible="no" active="yes"/>
@@
 <layer number="37" name="tTest" color="7" fill="1" visible="no" active="yes"/>
 <layer number="38" name="bTest" color="7" fill="1" visible="no" active="yes"/>
-<layer number="39" name="tKeepout" color="4" fill="11" visible="yes" active="yes"/>
-<layer number="40" name="bKeepout" color="1" fill="11" visible="yes" active="yes"/>
-<layer number="41" name="tRestrict" color="4" fill="10" visible="yes" active="yes"/>
-<layer number="42" name="bRestrict" color="1" fill="10" visible="yes" active="yes"/>
-<layer number="43" name="vRestrict" color="2" fill="10" visible="yes" active="yes"/>
-<layer number="44" name="Drills" color="7" fill="1" visible="yes" active="yes"/>
+<layer number="39" name="tKeepout" color="4" fill="11" visible="no" active="yes"/>
+<layer number="40" name="bKeepout" color="1" fill="11" visible="no" active="yes"/>
+<layer number="41" name="tRestrict" color="4" fill="10" visible="no" active="yes"/>
+<layer number="42" name="bRestrict" color="1" fill="10" visible="no" active="yes"/>
+<layer number="43" name="vRestrict" color="2" fill="10" visible="no" active="yes"/>
+<layer number="44" name="Drills" color="7" fill="1" visible="no" active="yes"/>
 <layer number="45" name="Holes" color="7" fill="1" visible="yes" active="yes"/>
 <layer number="46" name="Milling" color="3" fill="1" visible="yes" active="yes"/>
@@
 <text x="26.289" y="27.813" size="1.016" layer="21" ratio="20">+</text>
 <text x="21.971" y="27.94" size="0.6096" layer="21" ratio="20" rot="R90">GND</text>
-<text x="44.831" y="6.096" size="1.016" layer="21" ratio="20">LCD</text>
+<text x="42.037" y="6.096" size="1.016" layer="21" ratio="20">LCD</text>
 <text x="61.722" y="3.556" size="1.016" layer="21" ratio="20">JTAG</text>
 <text x="83.566" y="28.702" size="1.016" layer="21" ratio="20">PDI</text>
@@
 </class>
 </classes>
-<designrules name="FindMeSAT_MB_1V2">
+<designrules name="FindMeSAT_MB_1V2 *">
 <description language="de">&lt;p&gt;
 &lt;b&gt;Smart-Prototyping EAGLE design rules&lt;/b&gt;&lt;br&gt;
@@
 <wire x1="76.2" y1="10.58" x2="77.597" y2="9.906" width="0.1524" layer="16"/>
 <polygon width="0.4064" layer="15" rank="2">
-<vertex x="99.06" y="41.91"/>
+<vertex x="98.5" y="41.91"/>
 <vertex x="7.32" y="41.91"/>
-<vertex x="7.32" y="0"/>
-<vertex x="99.06" y="0"/>
+<vertex x="7.32" y="0.5"/>
+<vertex x="98.5" y="0.5"/>
 </polygon>
 <via x="57.785" y="29.845" extent="1-16" drill="0.3048" shape="octagon"/>
@@
 <wire x1="17.891" y1="40.37" x2="17.018" y2="41.402" width="0.254" layer="1"/>
 <wire x1="17.018" y1="41.402" x2="14.605" y2="41.402" width="0.254" layer="1"/>
-<contactref element="X121" pad="5"/>
-<contactref element="X121" pad="2"/>
 <contactref element="U301" pad="9"/>
 <contactref element="C301" pad="2"/>
@@
 <wire x1="41.91" y1="3.048" x2="42.545" y2="3.81" width="0.1524" layer="16"/>
 <wire x1="90.043" y1="6.604" x2="89.408" y2="6.604" width="0.1524" layer="1"/>
+<contactref element="X121" pad="1"/>
+<contactref element="X121" pad="6"/>
 <wire x1="89.408" y1="6.604" x2="89.084" y2="6.064" width="0" layer="19" extent="1-1"/>
 <wire x1="48.638590625" y1="18.64921875" x2="48.641" y2="18.634" width="0" layer="19" extent="1-1"/>
@@
 <wire x1="83.898" y1="37.26" x2="84.738" y2="38.1" width="0.254" layer="16"/>
 <wire x1="84.738" y1="38.1" x2="85.09" y2="38.1" width="0.15" layer="16"/>
-<contactref element="X121" pad="4"/>
-<wire x1="49.276" y1="6.477" x2="47.879" y2="7.874" width="0.4064" layer="16"/>
 <wire x1="47.879" y1="7.874" x2="44.069" y2="7.874" width="0.4064" layer="16"/>
 <wire x1="44.069" y1="7.874" x2="43.561" y2="8.382" width="0.4064" layer="16"/>
@@
 <wire x1="42.926" y1="26.543" x2="44.196" y2="27.813" width="0.4064" layer="1"/>
 <wire x1="83.898" y1="37.26" x2="83.82" y2="37.26" width="0.4064" layer="16"/>
+<contactref element="X121" pad="3"/>
+<wire x1="47.879" y1="7.874" x2="49.276" y2="6.477" width="0.4064" layer="16"/>
 </signal>
 <signal name="SW">
@@
 <wire x1="71.882" y1="10.033" x2="71.882" y2="8.89" width="0.1524" layer="16"/>
 <polygon width="0.4064" layer="2" rank="2">
-<vertex x="99.06" y="41.91"/>
+<vertex x="98.5" y="41.91"/>
 <vertex x="7.32" y="41.91"/>
-<vertex x="7.32" y="0"/>
-<vertex x="99.06" y="0"/>
+<vertex x="7.32" y="0.5"/>
+<vertex x="98.5" y="0.5"/>
 </polygon>
 <wire x1="61.026" y1="35.56" x2="61.126" y2="33.02" width="0.4064" layer="16"/>
@@
 <via x="46.482" y="10.668" extent="1-16" drill="0.3048" shape="octagon"/>
 <wire x1="45.593" y1="9.274" x2="46.358" y2="9.401" width="0.1524" layer="16"/>
-<contactref element="X121" pad="6"/>
 <wire x1="46.482" y1="9.528" x2="46.482" y2="10.668" width="0.1524" layer="16"/>
 <contactref element="U301" pad="8"/>
@@
 <wire x1="54.864" y1="17.907" x2="54.991" y2="18.034" width="0.1524" layer="1"/>
 <wire x1="54.991" y1="18.034" x2="54.991" y2="19.05" width="0.1524" layer="1"/>
+<contactref element="X121" pad="5"/>
 <wire x1="69.215" y1="18.288" x2="69.176" y2="18.288" width="0" layer="19" extent="16-16"/>
 <wire x1="54.571" y1="19.05" x2="54.991" y2="19.05" width="0" layer="19" extent="1-1"/>
@@
 <signal name="SDA2">
 <contactref element="U101" pad="16"/>
-<contactref element="X121" pad="3"/>
 <wire x1="63.373" y1="9.2456" x2="63.373" y2="8.128" width="0.1524" layer="1"/>
 <wire x1="63.373" y1="8.128" x2="63.373" y2="8.382" width="0.1524" layer="2"/>
@@
 <wire x1="54.61" y1="10.287" x2="53.721" y2="9.398" width="0.1524" layer="2"/>
 <wire x1="53.721" y1="9.398" x2="53.721" y2="8.382" width="0.1524" layer="2"/>
-<wire x1="53.721" y1="8.382" x2="51.816" y2="6.477" width="0.1524" layer="2"/>
 <via x="63.373" y="8.128" extent="1-16" drill="0.3048" shape="octagon"/>
+<contactref element="X121" pad="4"/>
+<wire x1="53.721" y1="8.382" x2="51.816" y2="6.477" width="0.1524" layer="2"/>
 </signal>
 <signal name="SCL2">
 <contactref element="U101" pad="17"/>
-<contactref element="X121" pad="1"/>
 <wire x1="65.1256" y1="7.493" x2="65.024" y2="7.3914" width="0.1524" layer="1"/>
 <wire x1="65.024" y1="7.3914" x2="65.024" y2="7.239" width="0.1524" layer="1"/>
@@
 <wire x1="51.308" y1="5.207" x2="50.546" y2="5.969" width="0.1524" layer="2"/>
 <wire x1="50.546" y1="5.969" x2="50.546" y2="7.747" width="0.1524" layer="2"/>
-<wire x1="50.546" y1="7.747" x2="51.816" y2="9.017" width="0.1524" layer="2"/>
 <via x="64.135" y="7.239" extent="1-16" drill="0.3048" shape="octagon"/>
+<contactref element="X121" pad="2"/>
+<wire x1="50.546" y1="7.747" x2="51.816" y2="9.017" width="0.1524" layer="2"/>
 </signal>
 <signal name="I2C2_INT">
