File: CAD/Eagle/FindMeSAT_MB_1V2.brd (EAGLE design)
At the start: 99 x 49.2 mm, 135 parts, among them Q101 ABS07-32.768KHZ, Q651 ABM3B-16MHZ-10-R50-1-U, U1001 CFPT-141-20MHZ, U101 ATXMEGA256A3BU-AU, U1011 OPA354, U1021 OPA354, U1111 LM2831YMF, U1121 LM4120IM5-3.0, U201 SIM808, U301 MPU-9250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

Commit message: HW_V1.2 - AX5243 UHF port - advanced values for matching unit / BALUN
Parts:
- C686: value 18pF -> 3.3pF
- L682: value 68nH -> 27nH
- L686: value 150nH -> 27nH
Changed lines of the file:
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@@
 <attribute name="VALUE" x="92.456" y="18.542" size="0.6096" layer="28" rot="MR0"/>
 </element>
-<element name="L686" library="rcl" package="R0603" value="150nH" x="89.027" y="9.144" smashed="yes" rot="MR90">
+<element name="L686" library="rcl" package="R0603" value="27nH" x="89.027" y="9.144" smashed="yes" rot="MR90">
 <attribute name="NAME" x="88.773" y="5.207" size="0.6096" layer="26" rot="MR90"/>
 <attribute name="VALUE" x="88.773" y="8.001" size="0.6096" layer="28" rot="MR90"/>
 </element>
-<element name="L682" library="rcl" package="R0603" value="68nH" x="94.742" y="16.256" smashed="yes" rot="MR270">
+<element name="L682" library="rcl" package="R0603" value="27nH" x="94.742" y="16.256" smashed="yes" rot="MR270">
 <attribute name="NAME" x="94.488" y="18.034" size="0.6096" layer="26" rot="MR90"/>
 <attribute name="VALUE" x="94.488" y="15.24" size="0.6096" layer="28" rot="MR90"/>
 </element>
-<element name="C686" library="rcl" package="C0603" value="18pF" x="94.742" y="10.668" smashed="yes" rot="MR90">
+<element name="C686" library="rcl" package="C0603" value="3.3pF" x="94.742" y="10.668" smashed="yes" rot="MR90">
 <attribute name="NAME" x="94.488" y="6.604" size="0.6096" layer="26" rot="MR90"/>
 <attribute name="VALUE" x="94.488" y="10.287" size="0.6096" layer="28" rot="MR90"/>

Commit message: HW_V1.2 - AX5243 UHF matching unit enhanced
Parts:
- C681: value 68pF -> 82pF
- C686: value 3.3pF -> 150pF
- L681: value 150nH -> 100nH
- L682: value 27nH -> 56nH
- L686: value 27nH -> 33nH
Changed lines of the file:
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@@
 <attribute name="VALUE" x="81.788" y="7.112" size="0.6096" layer="27"/>
 </element>
-<element name="C681" library="rcl" package="C0603" value="68pF" x="92.075" y="18.796" smashed="yes" rot="MR0">
+<element name="C681" library="rcl" package="C0603" value="82pF" x="92.075" y="18.796" smashed="yes" rot="MR0">
 <attribute name="NAME" x="93.345" y="19.685" size="0.6096" layer="26" rot="MR0"/>
 <attribute name="VALUE" x="92.456" y="18.542" size="0.6096" layer="28" rot="MR0"/>
 </element>
-<element name="L686" library="rcl" package="R0603" value="27nH" x="89.027" y="9.144" smashed="yes" rot="MR90">
+<element name="L686" library="rcl" package="R0603" value="33nH" x="89.027" y="9.144" smashed="yes" rot="MR90">
 <attribute name="NAME" x="88.773" y="5.207" size="0.6096" layer="26" rot="MR90"/>
 <attribute name="VALUE" x="88.773" y="8.001" size="0.6096" layer="28" rot="MR90"/>
 </element>
-<element name="L682" library="rcl" package="R0603" value="27nH" x="94.742" y="16.256" smashed="yes" rot="MR270">
+<element name="L682" library="rcl" package="R0603" value="56nH" x="94.742" y="16.256" smashed="yes" rot="MR270">
 <attribute name="NAME" x="94.488" y="18.034" size="0.6096" layer="26" rot="MR90"/>
 <attribute name="VALUE" x="94.488" y="15.24" size="0.6096" layer="28" rot="MR90"/>
 </element>
-<element name="C686" library="rcl" package="C0603" value="3.3pF" x="94.742" y="10.668" smashed="yes" rot="MR90">
+<element name="C686" library="rcl" package="C0603" value="150pF" x="94.742" y="10.668" smashed="yes" rot="MR90">
 <attribute name="NAME" x="94.488" y="6.604" size="0.6096" layer="26" rot="MR90"/>
 <attribute name="VALUE" x="94.488" y="10.287" size="0.6096" layer="28" rot="MR90"/>
 </element>
-<element name="L681" library="rcl" package="R0603" value="150nH" x="97.282" y="18.415" smashed="yes" rot="MR180">
+<element name="L681" library="rcl" package="R0603" value="100nH" x="97.282" y="18.415" smashed="yes" rot="MR180">
 <attribute name="NAME" x="98.425" y="19.304" size="0.6096" layer="26" rot="MR0"/>
 <attribute name="VALUE" x="98.552" y="18.161" size="0.6096" layer="28" rot="MR0"/>
