File: CAD/Eagle/FindMeSAT_MB_1V2.sch (EAGLE design)
At the start: 135 parts, among them Q101 ABS07-32.768KHZ, Q651 ABM3B-16MHZ-10-R50-1-U, U1001 CFPT-141-20MHZ, U101 ATXMEGA256A3BU-AU, U1011 OPA354, U1021 OPA354, U1111 LM2831YMF, U1121 LM4120IM5-3.0, U201 SIM808, U301 MPU-9250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

Commit message: HW_V1.2 - AX5243 UHF port - advanced values for matching unit / BALUN
Parts:
- C686: value 18pF -> 3.3pF
- L682: value 68nH -> 27nH
- L686: value 150nH -> 27nH
Changed lines of the file:
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@@
 <part name="C681" library="rcl" deviceset="C-EU" device="C0603" value="68pF"/>
 <part name="GND683" library="df4iah_supply" deviceset="GND" device=""/>
-<part name="L686" library="rcl" deviceset="R-EU_" device="R0603" value="150nH"/>
-<part name="L682" library="rcl" deviceset="R-EU_" device="R0603" value="68nH"/>
+<part name="L686" library="rcl" deviceset="R-EU_" device="R0603" value="27nH"/>
+<part name="L682" library="rcl" deviceset="R-EU_" device="R0603" value="27nH"/>
 <part name="GND684" library="df4iah_supply" deviceset="GND" device=""/>
-<part name="C686" library="rcl" deviceset="C-EU" device="C0603" value="18pF"/>
+<part name="C686" library="rcl" deviceset="C-EU" device="C0603" value="3.3pF"/>
 <part name="L681" library="rcl" deviceset="R-EU_" device="R0603" value="150nH"/>
 <part name="X685" library="df4iah_connector" deviceset="SMA_SMT_AMPHENOL-901-143" device="" value="SMA_CON"/>

Commit message: HW_V1.2 - AX5243 UHF matching unit enhanced
Parts:
- C681: value 68pF -> 82pF
- C686: value 3.3pF -> 150pF
- L681: value 150nH -> 100nH
- L682: value 27nH -> 56nH
- L686: value 27nH -> 33nH
Other:
- note added: "Add 150nH to GND here"
Changed lines of the file:
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@@
 <part name="Q651" library="df4iah_crystal" deviceset="ABM03B-16.000MHZ" device="" value="ABM3B-16MHZ-10-R50-1-U"/>
 <part name="L671" library="rcl" deviceset="R-EU_" device="R0603" value="22nH"/>
-<part name="C681" library="rcl" deviceset="C-EU" device="C0603" value="68pF"/>
+<part name="C681" library="rcl" deviceset="C-EU" device="C0603" value="82pF"/>
 <part name="GND683" library="df4iah_supply" deviceset="GND" device=""/>
-<part name="L686" library="rcl" deviceset="R-EU_" device="R0603" value="27nH"/>
-<part name="L682" library="rcl" deviceset="R-EU_" device="R0603" value="27nH"/>
+<part name="L686" library="rcl" deviceset="R-EU_" device="R0603" value="33nH"/>
+<part name="L682" library="rcl" deviceset="R-EU_" device="R0603" value="56nH"/>
 <part name="GND684" library="df4iah_supply" deviceset="GND" device=""/>
-<part name="C686" library="rcl" deviceset="C-EU" device="C0603" value="3.3pF"/>
-<part name="L681" library="rcl" deviceset="R-EU_" device="R0603" value="150nH"/>
+<part name="C686" library="rcl" deviceset="C-EU" device="C0603" value="150pF"/>
+<part name="L681" library="rcl" deviceset="R-EU_" device="R0603" value="100nH"/>
 <part name="X685" library="df4iah_connector" deviceset="SMA_SMT_AMPHENOL-901-143" device="" value="SMA_CON"/>
 <part name="GND689" library="df4iah_supply" deviceset="GND" device=""/>
@@
 <text x="121.92" y="119.38" size="1.778" layer="97">NC</text>
 <text x="121.92" y="109.22" size="1.778" layer="97">NC</text>
+<text x="203.2" y="50.8" size="1.778" layer="97" rot="R90">Add 150nH to GND here</text>
 </plain>
 <instances>
